Commit message: habilitados los pid, cambio de nombre de link para la base, cambio de nombre del recurso buscado en  xacro, cambio del launch

File: src/scorbot_tf/urdf/scorbot.urdf.xacro (robot description, xacro)
@@ -4,10 +4,10 @@
   name="scorbot">
   <!-- URDF Materials -->
-  <xacro:include filename="$(find scorbot_gazebo)/urdf/materials.urdf.xacro" />
+  <xacro:include filename="$(find scorbot_gazebo_tf)/urdf/materials.urdf.xacro" />
   <!-- Gazebo macros -->
-  <xacro:include filename="$(find scorbot_gazebo)/urdf/gazebo.urdf.xacro" />
+  <xacro:include filename="$(find scorbot_gazebo_tf)/urdf/gazebo.urdf.xacro" />
   <!-- Gazebo elements -->
   <!-- Gazebo Links material -->
-  <xacro:gazebo_dae_link link="base_" />
+  <xacro:gazebo_dae_link link="base_link" />
   <xacro:gazebo_dae_link link="body" />
   <xacro:gazebo_dae_link link="upper_arm" />
@@ -46,9 +46,9 @@
     <joint name="fixed" type="fixed">
       <parent link="world"/>
-      <child link="base_"/>
+      <child link="base_link"/>
     </joint>
   </xacro:if>
   <link
-    name="base_">
+    name="base_link">
     <inertial>
       <origin
@@ -71,5 +71,5 @@
       <geometry>
         <mesh
-          filename="package://scorbot_gazebo/meshes/base.dae" />
+          filename="package://scorbot_gazebo_tf/meshes/base.dae" />
       </geometry>
       <material
@@ -114,5 +114,5 @@
       <geometry>
         <mesh
-          filename="package://scorbot_gazebo/meshes/body.dae" />
+          filename="package://scorbot_gazebo_tf/meshes/body.dae" />
       </geometry>
       <material
@@ -136,5 +136,5 @@
       rpy="0 0 0" />
     <parent
-      link="base_" />
+      link="base_link" />
     <child
       link="body" />
@@ -165,5 +165,5 @@
       <geometry>
         <mesh
-          filename="package://scorbot_gazebo/meshes/upper_arm.dae" />
+          filename="package://scorbot_gazebo_tf/meshes/upper_arm.dae" />
       </geometry>
       <material
@@ -216,5 +216,5 @@
       <geometry>
         <mesh
-          filename="package://scorbot_gazebo/meshes/forearm.dae" />
+          filename="package://scorbot_gazebo_tf/meshes/forearm.dae" />
       </geometry>
       <material
@@ -267,5 +267,5 @@
       <geometry>
         <mesh
-          filename="package://scorbot_gazebo/meshes/flange.dae" />
+          filename="package://scorbot_gazebo_tf/meshes/flange.dae" />
       </geometry>
       <material
@@ -333,5 +333,5 @@
       <geometry>
         <mesh
-          filename="package://scorbot_gazebo/meshes/gripper_base.dae" />
+          filename="package://scorbot_gazebo_tf/meshes/gripper_base.dae" />
       </geometry>
       <material
@@ -376,5 +376,5 @@
       <geometry>
         <mesh
-          filename="package://scorbot_gazebo/meshes/gripper_finger.dae" />
+          filename="package://scorbot_gazebo_tf/meshes/gripper_finger.dae" />
       </geometry>
       <material
@@ -390,5 +390,5 @@
       <geometry>
         <mesh
-          filename="package://scorbot_gazebo/meshes/gripper_finger.dae" />
+          filename="package://scorbot_gazebo_tf/meshes/gripper_finger.dae" />
       </geometry>
     </collision>
@@ -430,5 +430,5 @@
       <geometry>
         <mesh
-          filename="package://scorbot_gazebo/meshes/gripper_finger.dae" />
+          filename="package://scorbot_gazebo_tf/meshes/gripper_finger.dae" />
       </geometry>
       <material
@@ -444,5 +444,5 @@
       <geometry>
         <mesh
-          filename="package://scorbot_gazebo/meshes/gripper_finger.dae" />
+          filename="package://scorbot_gazebo_tf/meshes/gripper_finger.dae" />
       </geometry>
     </collision>
