Commit message: tendría que ver que pasa si le doy más sleep al master...

File: modelo_scorbot_gazebo/src/scorbot_tf/urdf/scorbot.urdf (robot description, URDF)
Before this commit: robot scorbot, 8 links, 7 joints
Links:
- removed link base_
- added link base_link, mass 3.5594; collision cylinder length=0.045 radius=0.16; collision cylinder length=0.170 radius=0.05
- added link world
- link body: geometry collision box size=0.380 0.18 0.25; visual mesh filename=package://scorbot_gazebo_tf/meshes/body.dae
- link flange: geometry collision cylinder length=0.105 radius=0.05; visual mesh filename=package://scorbot_gazebo_tf/meshes/flange.dae
- link forearm: geometry collision box size=0.3 0.095 0.12; visual mesh filename=package://scorbot_gazebo_tf/meshes/forearm.dae
- link gripper_base_link: geometry collision box size=0.078 0.110 0.055; collision cylinder length=0.044 radius=0.05
- link gripper_finger_left: geometry collision mesh filename=package://scorbot_gazebo_tf/meshes/gripper_finger.dae; visual mesh filename=package://scorbot_gazebo_tf/meshes/gripper_finger.dae
- link gripper_finger_right: geometry collision mesh filename=package://scorbot_gazebo_tf/meshes/gripper_finger.dae; visual mesh filename=package://scorbot_gazebo_tf/meshes/gripper_finger.dae
- link upper_arm: geometry collision box size=0.60 0.12 0.16; visual mesh filename=package://scorbot_gazebo_tf/meshes/upper_arm.dae
Joints:
- added joint fixed: type fixed, parent world, child base_link
- joint base: axis 0 0 1 -> 0 0 -1; parent base_ -> base_link
- joint shoulder: axis 0 1 0 -> 0 -1 0
