Commit message: intentado modificar la simulacion para que se controle por posicion y velocidad. hay que ver trajectory controllers

File: modelo_scorbot_gazebo/src/scorbot_tf/urdf/gazebo.urdf.xacro (robot description, xacro)
@@ -31,4 +31,17 @@
       <actuator name="${joint}_motor">
         <hardwareInterface>hardware_interface/PositionJointInterface</hardwareInterface>
+        <mechanicalReduction>1</mechanicalReduction>
+      </actuator>
+    </transmission>
+  </xacro:macro>
+  <!-- For Velocity controllers -->
+  <xacro:macro name="joint_vel_transmission" params="joint">
+    <transmission name="${joint}_transmission">
+      <type>transmission_interface/SimpleTransmission</type>
+      <joint name="${joint}">
+       <hardwareInterface>hardware_interface/VelocityJointInterface</hardwareInterface>
+      </joint>
+      <actuator name="${joint}_motor">
+        <hardwareInterface>hardware_interface/VelocityJointInterface</hardwareInterface>
         <mechanicalReduction>1</mechanicalReduction>
       </actuator>
