Commit message: recuperacion de scorbot.urdf y ahora corre el Scorbot_7_moveit.urdf

File: software_scorbot/scorbot_catkin_ws/src/scorbot_7_moveit/modelo/Scorbot_7.urdf (robot description, URDF)
Before this commit: robot Scorbot_7, 11 links, 10 joints
Links:
- link base_link: geometry visual mesh filename=package://scorbot_7_moveit/modelo/base_robot.dae scale=1 1 1
- link link1: geometry visual mesh filename=package://scorbot_7_moveit/modelo/link1.dae scale=1 1 1
- link link2: geometry visual mesh filename=package://scorbot_7_moveit/modelo/link2.dae scale=1 1 1
- link link3: geometry visual mesh filename=package://scorbot_7_moveit/modelo/link3.dae scale=1 1 1
- link link4: geometry visual mesh filename=package://scorbot_7_moveit/modelo/link4.dae scale=1 1 1
- link link5: geometry visual mesh filename=package://scorbot_7_moveit/modelo/link5.dae scale=1 1 1
- link table: geometry visual mesh filename=package://scorbot_7_moveit/modelo/mesa.dae scale=1 1 1
