Commit message: intento de hacer que funcionen los controles para gazebo. Habría que ver la versión completa del panda y comparar como están hechos ahí

File: software_scorbot/scorbot_catkin_ws/src/scorbot_gazebo_tf/urdf/scorbot.urdf.xacro (robot description, xacro)
@@ -57,5 +57,5 @@
     </xacro:if>
 -->
-<!--
+    <xacro:arg name="fixed" default="true"/>
     <xacro:if value="$(arg fixed)">
     <link name="world"/>
@@ -65,5 +65,4 @@
     </joint>
   </xacro:if>
--->
   <link
     name="base_link">

File: software_scorbot/scorbot_catkin_ws/src/scorbot_vii_moveit/config/gazebo_scorbot.urdf (robot description, URDF)
Before this commit: robot scorbot, 8 links, 7 joints
Links:
- added link world
Joints:
- added joint fixed: type fixed, parent world, child base_link
